Commit message: add the fsm, arm controller, mirte_msgs, mirte_navigation proj_pts_location pkgs

File: arm_controller/config/arm.xacro (robot description, xacro)
@@ -1,4 +1,11 @@
 <?xml version="1.0" encoding="UTF-8"?>
-<robot xmlns:xacro="http://www.ros.org/wiki/xacro">
+<robot xmlns:xacro="http://www.ros.org/wiki/xacro" name="arm">
+    <link name="base_link"/>
+    <link name="frame_link"/>
+    <joint name="frame_base_joint" type="fixed">
+    <origin xyz="0 0 0.10" rpy="0 0 ${radians(90)}" />
+    <parent link="base_link" />
+    <child link="frame_link" />
+  </joint>
     <link
         name="shoulder_pan">
